File: pico-rgbi-to-vga.kicad_pcb (KiCad board)
At the start: 2 copper layers, 68.8 x 57 mm, 28 parts, among them J1 SDS-80J, J2 DB15_Female_HighDensity, J3 USB-B1HSB6, Q1 2n2222, Q2 2n2222, SW1 SW_Push, U1 Pico

Commit message: Palette toggle button
Other:
- board text added: "PC-6001 Forever"
Changed lines of the file:
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@@
   (gr_arc (start 162 63) (mid 167.656854 65.343146) (end 170 71) (layer "Edge.Cuts") (width 0.1))
   (gr_line (start 170 71) (end 170 112) (layer "Edge.Cuts") (width 0.1))
+  (gr_text "PC-6001 Forever" (at 145.796 91.735001 90) (layer "B.Cu")
+    (effects (font (size 1.5 1.5) (thickness 0.3)) (justify mirror))
+  )
   (gr_text "Pin 3" (at 109.169 69.69) (layer "F.SilkS")
     (effects (font (size 1 1) (thickness 0.15)))

Commit message: V0.1 sent to Fab
Other:
- board text added: "Q1, Q2 = 2n2222"
