File: pico-rgbi-to-vga.kicad_sch (KiCad schematic)
At the start: 25 parts, among them J1 SDS-80J, J2 DB15_Female_HighDensity, J3 USB-B1HSB6, SW1 SW_Push, SW2 Intensity Select, U1 Pico

Commit message: KiCad7; reorder pins so HV won't get captured
Connections:
- net BLUE_3v3: now also U1.2 (GPIO1); no longer U1.5 (GPIO3)
- net GREEN_3v3: now also U1.4 (GPIO2); no longer U1.6 (GPIO4)
- net HSYNC_3v3: no longer U1.4 (GPIO2)
- net RED_3v3: now also U1.5 (GPIO3); no longer U1.7 (GPIO5)
- net VSYNC_3v3: now also U1.6 (GPIO4); no longer U1.2 (GPIO1)
